Commit message: Adding welding tools

File: ur_description_pkg/ur_description/urdf/ur10.urdf.xacro (robot description, xacro)
@@ -336,4 +336,100 @@
       <child link="${prefix}tool0"/>
     </joint>
+    <!-- *************************************************** -->
+ <link name="torch">
+	<visual name="visual">
+      <geometry>
+        <mesh filename="package://ppm_lab/meshes/torch.stl"/>
+      </geometry>
+      <material name="red"/>
+      <!-- <material name="torch_gray"/> -->
+    </visual>
+  </link>
+        <link name="tcp">
+	  <visual name="visual">
+      <geometry>
+        <sphere radius="0.005"/>
+      </geometry>
+    <material name="red"/>
+    </visual>
+  </link>
+  <link name="tip">
+	  <visual name="visual">
+      <geometry>
+        <sphere radius="0.005"/>
+      </geometry>
+      <!-- <material name="blue"/> -->
+    </visual>
+  </link>
+  <link name="scanner">
+	<visual name="visual">
+      <geometry>
+        <sphere radius="0.005"/>
+      </geometry>
+      <!-- <material name="red"/> -->
+    </visual>
+  </link>
+  <!-- <link name="table">
+	<visual name="visual">
+      <geometry>
+        <mesh filename="package://ppm_lab/meshes/table.stl"/>
+      </geometry>
+      <material name="desk_dark"/>
+    </visual>
+  </link> -->
+  <!-- <link name="plate">
+	  <visual name="visual">
+      <geometry>
+        <mesh filename="package://ppm_lab/meshes/workpiece.stl"/>
+      </geometry>
+      <material name="plate_light_gray"/>
+    </visual>
+  </link> -->
+  <link name="flange">
+	  <visual name="visual">
+      <geometry>
+        <mesh filename="package://ppm_lab/meshes/flange.stl"
+	      scale="0.001 0.001 0.001"/>
+      </geometry>
+      <!-- <material name="plate_light_gray"/> -->
+      <!-- <material name="blue"/> -->
+    </visual>
+  </link>
+ <joint type="fixed" name="link6_flange">
+    <origin xyz="0 0 0" rpy="1.570796 0 1.570796"/>
+        <!-- <origin xyz=" 0 0 0" rpy="0 0 0"/> -->
+    <parent link="${prefix}ee_link"/>
+    <child link="flange"/>
+    <!-- <axis xyz="0 1 0"/> -->
+  </joint>
+  <joint type="fixed" name="flange_torch">
+    <origin xyz="0.101 0.131 -0.006" rpy="0 0 1.570796"/>
+    <parent link="flange"/>
+    <child link="torch"/>
+    <axis xyz="0 0 1"/>
+  </joint>
+    <joint type="revolute" name="torch_tip">
+    <origin xyz="0.4295 0 0" rpy="0 -0.785398 0"/>
+    <parent link="${prefix}ee_link"/>
+    <child link="tip"/>
+    <axis xyz="0 0 1"/>
+    <limit lower="0" upper="0" effort="0" velocity="0"/>
+  </joint>
+      <joint type="revolute" name="scanner_tip">
+    <origin xyz="0.313575 0.059613 -0.03619" rpy="0.785398 0 -1.570796"/>
+    <parent link="${prefix}ee_link"/>
+    <child link="scanner"/>
+    <axis xyz="1 0 0"/>
+    <limit lower="0" upper="0" effort="0" velocity="0"/>
+  </joint>
+    <joint type="revolute" name="link_6_tcp">
+    <origin xyz=" 0 0 0" rpy="0 0 0"/>
+    <parent link="${prefix}ee_link"/>
+    <child link="tcp"/>
+    <!-- <origin xyz="0 0 0"/> -->
+    <!-- <axis xyz="0 0 1"/> -->
+    <limit lower="0" upper="0" effort="0" velocity="0"/>
+  </joint>
+    <!-- *************************************************** -->
   </xacro:macro>
 </robot>

Commit message: Modified URDF to use weld tool directly

File: ur_description_pkg/ur_description/urdf/ur10.urdf.xacro (robot description, xacro)
@@ -340,5 +340,5 @@
 	<visual name="visual">
       <geometry>
-        <mesh filename="package://ppm_lab/meshes/torch.stl"/>
+        <mesh filename="package://ur_description_pkg/ur_description/meshes/collision/torch.stl"/>
       </geometry>
       <material name="red"/>
@@ -370,24 +370,8 @@
     </visual>
   </link>
-  <!-- <link name="table">
-	<visual name="visual">
-      <geometry>
-        <mesh filename="package://ppm_lab/meshes/table.stl"/>
-      </geometry>
-      <material name="desk_dark"/>
-    </visual>
-  </link> -->
-  <!-- <link name="plate">
-	  <visual name="visual">
-      <geometry>
-        <mesh filename="package://ppm_lab/meshes/workpiece.stl"/>
-      </geometry>
-      <material name="plate_light_gray"/>
-    </visual>
-  </link> -->
   <link name="flange">
 	  <visual name="visual">
       <geometry>
-        <mesh filename="package://ppm_lab/meshes/flange.stl"
+        <mesh filename="package://ur_description_pkg/ur_description/meshes/collision/flange.stl"
 	      scale="0.001 0.001 0.001"/>
       </geometry>

Commit message: Modify tip position

File: ur_description_pkg/ur_description/urdf/ur10.urdf.xacro (robot description, xacro)
@@ -342,7 +342,14 @@
         <mesh filename="package://ur_description_pkg/ur_description/meshes/collision/torch.stl"/>
       </geometry>
-      <material name="red"/>
+      <material name="torch_gray"/>
       <!-- <material name="torch_gray"/> -->
     </visual>
+    <!--
+    <collision>
+        <geometry>
+          <mesh filename="package://ur_description_pkg/ur_description/meshes/collision/torch.stl"/>
+        </geometry>
+    </collision>
+    -->
   </link>
         <link name="tcp">
@@ -351,5 +358,5 @@
         <sphere radius="0.005"/>
       </geometry>
-    <material name="red"/>
+    <material name="torch_gray"/>
     </visual>
   </link>
@@ -359,5 +366,5 @@
         <sphere radius="0.005"/>
       </geometry>
-      <!-- <material name="blue"/> -->
+      <material name="blue"/>
     </visual>
   </link>
@@ -367,5 +374,5 @@
         <sphere radius="0.005"/>
       </geometry>
-      <!-- <material name="red"/> -->
+      <material name="torch_gray"/>
     </visual>
   </link>
@@ -376,7 +383,14 @@
 	      scale="0.001 0.001 0.001"/>
       </geometry>
-      <!-- <material name="plate_light_gray"/> -->
+      <material name="plate_light_gray"/>
       <!-- <material name="blue"/> -->
     </visual>
+    <!--
+    <collision>
+        <geometry>
+          <mesh filename="package://ur_description_pkg/ur_description/meshes/collision/flange.stl"/>
+        </geometry>
+    </collision>
+      -->
   </link>
  <joint type="fixed" name="link6_flange">
@@ -394,5 +408,6 @@
   </joint>
     <joint type="revolute" name="torch_tip">
-    <origin xyz="0.4295 0 0" rpy="0 -0.785398 0"/>
+    <!--<origin xyz="0.4295 0 0" rpy="0 -0.785398 0"/> -->
+    <origin xyz="0.38 0 0" rpy="0 -0.785398 0"/>
     <parent link="${prefix}ee_link"/>
     <child link="tip"/>

Commit message: Commit to pull

File: ur_description_pkg/ur_description/urdf/ur10.urdf.xacro (robot description, xacro)
@@ -342,5 +342,7 @@
         <mesh filename="package://ur_description_pkg/ur_description/meshes/collision/torch.stl"/>
       </geometry>
-      <material name="red"/>
+      <material name="LightGrey">
+               <color rgba="0.7 0.7 0.7 1.0"/>
+            </material>
       <!-- <material name="torch_gray"/> -->
     </visual>
@@ -351,5 +353,7 @@
         <sphere radius="0.005"/>
       </geometry>
-    <material name="red"/>
+    <material name="LightGrey">
+               <color rgba="0.7 0.7 0.7 1.0"/>
+            </material>
     </visual>
   </link>
@@ -376,4 +380,7 @@
 	      scale="0.001 0.001 0.001"/>
       </geometry>
+      <material name="LightGrey">
+               <color rgba="0.7 0.7 0.7 1.0"/>
+            </material>
       <!-- <material name="plate_light_gray"/> -->
       <!-- <material name="blue"/> -->

Commit message: Change tourch and flange color and add collision

File: ur_description_pkg/ur_description/urdf/ur10.urdf.xacro (robot description, xacro)
@@ -342,8 +342,9 @@
         <mesh filename="package://ur_description_pkg/ur_description/meshes/collision/torch.stl"/>
       </geometry>
-      <material name="torch_gray"/>
+      <material name="gunmetal_gray">
+        <color rgba="0.553 0.569 0.553 1.0"/>
+      </material>
       <!-- <material name="torch_gray"/> -->
     </visual>
-    <!--
     <collision>
         <geometry>
@@ -351,5 +352,4 @@
         </geometry>
     </collision>
-    -->
   </link>
         <link name="tcp">
@@ -358,5 +358,7 @@
         <sphere radius="0.005"/>
       </geometry>
-    <material name="torch_gray"/>
+    <material name="gunmetal_gray">
+        <color rgba="0.553 0.569 0.553 1.0"/>
+    </material>
     </visual>
   </link>
@@ -366,5 +368,7 @@
         <sphere radius="0.005"/>
       </geometry>
-      <material name="blue"/>
+      <material name="blue">
+        <color rgba="0 0 1 1.0"/>
+      </material>
     </visual>
   </link>
@@ -374,5 +378,7 @@
         <sphere radius="0.005"/>
       </geometry>
-      <material name="torch_gray"/>
+      <material name="gunmetal_gray">
+        <color rgba="0.553 0.569 0.553 1.0"/>
+      </material>
     </visual>
   </link>
@@ -383,6 +389,7 @@
 	      scale="0.001 0.001 0.001"/>
       </geometry>
-      <material name="plate_light_gray"/>
-      <!-- <material name="blue"/> -->
+      <material name="pewter">
+        <color rgba="0.914 0.918 0.925 1.0"/>
+      </material>
     </visual>
     <!--
